Commit message: enabled cameras of simulated drones. Removed the dedicated topic for the DRL contoller. Renamed the ros-topics of cameras

File: src/sim_ardrone/src/cvg_sim_gazebo/urdf/quadrotor_sensors.urdf.xacro (robot description, xacro)
@@ -16,5 +16,5 @@
     </xacro:sonar_sensor>
     <xacro:include filename="$(find cvg_sim_gazebo)/urdf/sensors/lidar_sensor.urdf.xacro" />
-    <xacro:lidar_sensor name="lidar" parent="base_link" ros_topic="lidar_collision" update_rate="10" min_range="0.1" max_range="5.0" field_of_view_h="${180*M_PI/180}" field_of_view_v="${1*M_PI/180}" ray_count_h="360" ray_count_v="1">
+    <xacro:lidar_sensor name="lidar" parent="base_link" ros_topic="scan" update_rate="10" min_range="0.2" max_range="2.0" field_of_view_h="${360*M_PI/180}" field_of_view_v="${1*M_PI/180}" ray_count_h="180" ray_count_v="1">
       <origin xyz="0.0 0.0 0.1" rpy="0 0 0"/>
     </xacro:lidar_sensor>
@@ -26,12 +26,12 @@
     <!-- The following two cameras should be united to one! -->
     <!-- Forward facing camera -->
-    <!--<xacro:include filename="$(find cvg_sim_gazebo)/urdf/sensors/generic_camera.urdf.xacro" />
-    <xacro:generic_camera name="front" sim_name="ardrone" parent="base_link" update_rate="60" res_x="640" res_y="360" image_format="R8G8B8" hfov="${81*M_PI/180}">
+    <xacro:include filename="$(find cvg_sim_gazebo)/urdf/sensors/generic_camera.urdf.xacro" />
+    <xacro:generic_camera name="front" parent="base_link" update_rate="60" res_x="640" res_y="360" image_format="R8G8B8" hfov="${81*M_PI/180}">
       <origin xyz="0.21 0.0 0.01" rpy="0 0 0"/>
-    </xacro:generic_camera>-->
+    </xacro:generic_camera>
     <!-- Downward facing camera -->
-    <!--<xacro:include filename="$(find cvg_sim_gazebo)/urdf/sensors/generic_camera.urdf.xacro" />
-    <xacro:generic_camera name="bottom" sim_name="ardrone" parent="base_link" update_rate="60" res_x="640" res_y="360" image_format="R8G8B8" hfov="${81*M_PI/180}">
+    <xacro:include filename="$(find cvg_sim_gazebo)/urdf/sensors/generic_camera.urdf.xacro" />
+    <xacro:generic_camera name="bottom" parent="base_link" update_rate="60" res_x="640" res_y="360" image_format="R8G8B8" hfov="${81*M_PI/180}">
       <origin xyz="0.15 0.0 0.0" rpy="0 ${M_PI/2} 0"/>
-    </xacro:generic_camera>-->
+    </xacro:generic_camera>
 </robot>

File: src/sim_ardrone/src/cvg_sim_gazebo/urdf/sensors/generic_camera.urdf.xacro (robot description, xacro)
@@ -6,5 +6,5 @@
   >
     <property name="M_PI" value="3.1415926535897931" />
-    <xacro:macro name="generic_camera" params="name sim_name parent *origin update_rate res_x res_y image_format hfov">
+    <xacro:macro name="generic_camera" params="name parent *origin update_rate res_x res_y image_format hfov">
       <joint name="${name}_joint" type="fixed">
         <insert_block name="origin" />
@@ -23,7 +23,7 @@
             <box size="0.01 0.01 0.01" />
           </geometry>
-	  <material name="Blue">
-      <color rgba="0.0 0.0 0.8 1"/>
-    </material>
+    	  <material name="Blue">
+          <color rgba="0.0 0.0 0.8 1"/>
+        </material>
         </visual>
         <collision>
@@ -71,14 +71,14 @@
           </image>
           <clip>0.01
-	    <near>0.01</near>
+	         <near>0.01</near>
             <far>100</far>
           </clip>
         </camera>
         <plugin name="${name}_camera_controller" filename="libgazebo_ros_camera.so">
-	  <cameraName>/${sim_name}/${name}</cameraName>
+	      <cameraName>${name}</cameraName>
           <alwaysOn>true</alwaysOn>
           <updateRate>${update_rate}</updateRate>
-          <imageTopicName>${sim_name}/${name}/image_raw</imageTopicName>
-          <cameraInfoTopicName>${sim_name}/${name}/camera_info</cameraInfoTopicName>
+          <imageTopicName>image_raw</imageTopicName>
+          <cameraInfoTopicName>camera_info</cameraInfoTopicName>
           <frameName>ardrone_base_${name}cam</frameName>
         </plugin>

File: src/sim_ardrone/src/cvg_sim_gazebo_plugins/urdf/quadrotor_sensors.urdf.xacro (robot description, xacro)
@@ -15,5 +15,5 @@
         <bodyName>base_link</bodyName>
         <frameId>ardrone_base_link</frameId>
-        <topicName>ardrone/imu</topicName>
+        <topicName>imu</topicName>
         <rpyOffsets>0 0 0</rpyOffsets> <!-- deprecated -->
         <gaussianNoise>0</gaussianNoise>  <!-- deprecated -->
@@ -23,10 +23,10 @@
         <rateGaussianNoise>0.00 0.00 0.00</rateGaussianNoise>
         <headingDrift>0.0</headingDrift>
-	<headingDriftFrequency>0.0</headingDriftFrequency>
-	<headingOffset>0.0	</headingOffset>
-	<rateDriftFrequency>0 0 0</rateDriftFrequency>
-	<rateOffset>0 0 0</rateOffset>
-	<accelDriftFrequency>0 0 0</accelDriftFrequency>
-	<accelOffset>0 0 0</accelOffset>
+      	<headingDriftFrequency>0.0</headingDriftFrequency>
+      	<headingOffset>0.0	</headingOffset>
+      	<rateDriftFrequency>0 0 0</rateDriftFrequency>
+      	<rateOffset>0 0 0</rateOffset>
+      	<accelDriftFrequency>0 0 0</accelDriftFrequency>
+      	<accelOffset>0 0 0</accelOffset>
         <headingGaussianNoise>0.00</headingGaussianNoise>
       </plugin>
@@ -39,5 +39,5 @@
         <offset>0</offset>
         <drift>0.1</drift>
-	<driftFrequency>0.0</driftFrequency>
+        <driftFrequency>0.0</driftFrequency>
         <gaussianNoise>0.5</gaussianNoise>
       </plugin>
@@ -49,5 +49,5 @@
         <offset>0 0 0</offset>
         <drift>0.0 0.0 0.0</drift>
-	<driftFrequency>0.0 0.0 0.0</driftFrequency>
+        <driftFrequency>0.0 0.0 0.0</driftFrequency>
         <gaussianNoise>1.3e-2 1.3e-2 1.3e-2</gaussianNoise>
       </plugin>
@@ -58,12 +58,12 @@
         <topicName>fix</topicName>
         <velocityTopicName>fix_velocity</velocityTopicName>
-	<offset>0 0 0</offset>
+      	<offset>0 0 0</offset>
         <drift>5.0 5.0 5.0</drift>
-	<driftFrequency>0.0 0.0 0.0</driftFrequency>
+      	<driftFrequency>0.0 0.0 0.0</driftFrequency>
         <gaussianNoise>0.1 0.1 0.1</gaussianNoise>
         <velocityDrift>0 0 0</velocityDrift>
         <velocityDriftFrequency>0 0 0</velocityDriftFrequency>
         <velocityGaussianNoise>0.1 0.1 0.1</velocityGaussianNoise>
-	<velocityOffset>0 0 0</velocityOffset>
+      	<velocityOffset>0 0 0</velocityOffset>
       </plugin>
       <plugin name="quadrotor_groundtruth_sim" filename="libgazebo_ros_p3d.so">

File: src/sim_ardrone/src/cvg_sim_gazebo_plugins/urdf/quadrotor_simple_controller.urdf.xacro (robot description, xacro)
@@ -12,5 +12,5 @@
         <bodyName>base_link</bodyName>
         <stateTopic>ground_truth/state</stateTopic>
-        <imuTopic>ardrone/imu</imuTopic>
+        <imuTopic>imu</imuTopic>
         <topicName>cmd_vel</topicName>
         <rollpitchProportionalGain>10.0</rollpitchProportionalGain>
@@ -36,7 +36,7 @@
         <bodyName>base_link</bodyName>
         <stateTopic>ground_truth/state</stateTopic>
-        <imuTopic>ardrone/imu</imuTopic>
+        <imuTopic>imu</imuTopic>
         <sonarTopic>sonar_height</sonarTopic>
-        <lidarTopic>lidar_collision</lidarTopic>
+        <lidarTopic>scan</lidarTopic>
         <topicName>cmd_vel</topicName>
       </plugin>

Commit message: added ddpg_networks with various lstm config

File: src/sim_ardrone/src/cvg_sim_gazebo/urdf/quadrotor_sensors.urdf.xacro (robot description, xacro)
@@ -16,6 +16,6 @@
     </xacro:sonar_sensor>
     <xacro:include filename="$(find cvg_sim_gazebo)/urdf/sensors/lidar_sensor.urdf.xacro" />
-    <xacro:lidar_sensor name="lidar" parent="base_link" ros_topic="scan" update_rate="10" min_range="0.2" max_range="2.0" field_of_view_h="${360*M_PI/180}" field_of_view_v="${1*M_PI/180}" ray_count_h="180" ray_count_v="1">
-      <origin xyz="0.0 0.0 0.1" rpy="0 0 0"/>
+    <xacro:lidar_sensor name="lidar" parent="base_link" ros_topic="scan" update_rate="10" min_range="0.35" max_range="2.0" field_of_view_h="${360*M_PI/180}" field_of_view_v="${1*M_PI/180}" ray_count_h="180" ray_count_v="1">
+      <origin xyz="0.0 0.0 0.025" rpy="0 0 0"/>
     </xacro:lidar_sensor>
     <!-- Hokuyo UTM-30LX mounted upside down below the quadrotor body

File: src/sim_ardrone/src/cvg_sim_gazebo/urdf/sensors/lidar_sensor.urdf.xacro (robot description, xacro)
@@ -13,13 +13,12 @@
     <link name="${name}_link">
       <inertial>
-        <mass value="0.001" />
+        <mass value="0.0" />
         <origin xyz="0 0 0" rpy="0 0 0" />
-        <inertia ixx="0.000000017" ixy="0" ixz="0" iyy="0.000000017" iyz="0" izz="0.000000017" />
+        <inertia ixx="0.0" ixy="0" ixz="0" iyy="0.0" iyz="0" izz="0.0" />
       </inertial>
       <visual>
         <origin xyz="0 0 0" rpy="0 0 0" />
         <geometry>
-          <box size="0.1 0.1 0.2" />
-          <!--<mesh filename="package://cvg_sim_gazebo/meshes/sonar_sensor/max_sonar_ez4.dae"/>-->
+          <mesh filename="package://cvg_sim_gazebo/meshes/sonar_sensor/max_sonar_ez4.dae"/>
         </geometry>
       </visual>
@@ -27,5 +26,5 @@
         <origin xyz="0 0 0" rpy="0 0 0" />
         <geometry>
-          <box size="0.1 0.1 0.2" />
+          <box size="0.0 0.0 0.0" />
         </geometry>
       </collision>
@@ -63,5 +62,5 @@
           <offset>0.0 </offset>
           <drift>0.0</drift>
-	  <driftFrequency>0.0</driftFrequency>
+          <driftFrequency>0.0</driftFrequency>
           <topicName>${ros_topic}</topicName>
           <frameId>${name}_link</frameId>

Commit message: added logs, revised paramters

File: src/sim_ardrone/src/cvg_sim_gazebo/urdf/quadrotor_sensors.urdf.xacro (robot description, xacro)
@@ -16,6 +16,6 @@
     </xacro:sonar_sensor>
     <xacro:include filename="$(find cvg_sim_gazebo)/urdf/sensors/lidar_sensor.urdf.xacro" />
-    <xacro:lidar_sensor name="lidar" parent="base_link" ros_topic="scan" update_rate="10" min_range="0.35" max_range="5.0" field_of_view_h="${180*M_PI/180}" field_of_view_v="${1*M_PI/180}" ray_count_h="180" ray_count_v="1">
-      <origin xyz="0.0 0.0 0.025" rpy="0 0 0"/>
+    <xacro:lidar_sensor name="lidar" parent="base_link" ros_topic="lidar_collision" update_rate="10" min_range="0.1" max_range="5.0" field_of_view_h="${180*M_PI/180}" field_of_view_v="${1*M_PI/180}" ray_count_h="180" ray_count_v="1">
+      <origin xyz="0.0 0.0 0.1" rpy="0 0 0"/>
     </xacro:lidar_sensor>
     <!-- Hokuyo UTM-30LX mounted upside down below the quadrotor body
@@ -26,12 +26,12 @@
     <!-- The following two cameras should be united to one! -->
     <!-- Forward facing camera -->
-    <xacro:include filename="$(find cvg_sim_gazebo)/urdf/sensors/generic_camera.urdf.xacro" />
-    <xacro:generic_camera name="front" parent="base_link" update_rate="60" res_x="640" res_y="360" image_format="R8G8B8" hfov="${81*M_PI/180}">
+    <!--<xacro:include filename="$(find cvg_sim_gazebo)/urdf/sensors/generic_camera.urdf.xacro" />
+    <xacro:generic_camera name="front" sim_name="ardrone" parent="base_link" update_rate="60" res_x="640" res_y="360" image_format="R8G8B8" hfov="${81*M_PI/180}">
       <origin xyz="0.21 0.0 0.01" rpy="0 0 0"/>
-    </xacro:generic_camera>
+    </xacro:generic_camera>-->
     <!-- Downward facing camera -->
-    <xacro:include filename="$(find cvg_sim_gazebo)/urdf/sensors/generic_camera.urdf.xacro" />
-    <xacro:generic_camera name="bottom" parent="base_link" update_rate="60" res_x="640" res_y="360" image_format="R8G8B8" hfov="${81*M_PI/180}">
+    <!--<xacro:include filename="$(find cvg_sim_gazebo)/urdf/sensors/generic_camera.urdf.xacro" />
+    <xacro:generic_camera name="bottom" sim_name="ardrone" parent="base_link" update_rate="60" res_x="640" res_y="360" image_format="R8G8B8" hfov="${81*M_PI/180}">
       <origin xyz="0.15 0.0 0.0" rpy="0 ${M_PI/2} 0"/>
-    </xacro:generic_camera>
+    </xacro:generic_camera>-->
 </robot>

File: src/sim_ardrone/src/cvg_sim_gazebo/urdf/sensors/generic_camera.urdf.xacro (robot description, xacro)
@@ -6,5 +6,5 @@
   >
     <property name="M_PI" value="3.1415926535897931" />
-    <xacro:macro name="generic_camera" params="name parent *origin update_rate res_x res_y image_format hfov">
+    <xacro:macro name="generic_camera" params="name sim_name parent *origin update_rate res_x res_y image_format hfov">
       <joint name="${name}_joint" type="fixed">
         <insert_block name="origin" />
@@ -23,7 +23,7 @@
             <box size="0.01 0.01 0.01" />
           </geometry>
-    	  <material name="Blue">
-          <color rgba="0.0 0.0 0.8 1"/>
-        </material>
+	  <material name="Blue">
+      <color rgba="0.0 0.0 0.8 1"/>
+    </material>
         </visual>
         <collision>
@@ -71,14 +71,14 @@
           </image>
           <clip>0.01
-	         <near>0.01</near>
+	    <near>0.01</near>
             <far>100</far>
           </clip>
         </camera>
         <plugin name="${name}_camera_controller" filename="libgazebo_ros_camera.so">
-	      <cameraName>${name}</cameraName>
+	  <cameraName>/${sim_name}/${name}</cameraName>
           <alwaysOn>true</alwaysOn>
           <updateRate>${update_rate}</updateRate>
-          <imageTopicName>image_raw</imageTopicName>
-          <cameraInfoTopicName>camera_info</cameraInfoTopicName>
+          <imageTopicName>${sim_name}/${name}/image_raw</imageTopicName>
+          <cameraInfoTopicName>${sim_name}/${name}/camera_info</cameraInfoTopicName>
           <frameName>ardrone_base_${name}cam</frameName>
         </plugin>

File: src/sim_ardrone/src/cvg_sim_gazebo/urdf/sensors/lidar_sensor.urdf.xacro (robot description, xacro)
@@ -13,12 +13,13 @@
     <link name="${name}_link">
       <inertial>
-        <mass value="0.0" />
+        <mass value="0.001" />
         <origin xyz="0 0 0" rpy="0 0 0" />
-        <inertia ixx="0.0" ixy="0" ixz="0" iyy="0.0" iyz="0" izz="0.0" />
+        <inertia ixx="0.000000017" ixy="0" ixz="0" iyy="0.000000017" iyz="0" izz="0.000000017" />
       </inertial>
       <visual>
         <origin xyz="0 0 0" rpy="0 0 0" />
         <geometry>
-          <mesh filename="package://cvg_sim_gazebo/meshes/sonar_sensor/max_sonar_ez4.dae"/>
+          <box size="0.1 0.1 0.2" />
+          <!--<mesh filename="package://cvg_sim_gazebo/meshes/sonar_sensor/max_sonar_ez4.dae"/>-->
         </geometry>
       </visual>
@@ -26,5 +27,5 @@
         <origin xyz="0 0 0" rpy="0 0 0" />
         <geometry>
-          <box size="0.0 0.0 0.0" />
+          <box size="0.1 0.1 0.2" />
         </geometry>
       </collision>
@@ -62,5 +63,5 @@
           <offset>0.0 </offset>
           <drift>0.0</drift>
-          <driftFrequency>0.0</driftFrequency>
+	  <driftFrequency>0.0</driftFrequency>
           <topicName>${ros_topic}</topicName>
           <frameId>${name}_link</frameId>

File: src/sim_ardrone/src/cvg_sim_gazebo_plugins/urdf/quadrotor_sensors.urdf.xacro (robot description, xacro)
@@ -15,5 +15,5 @@
         <bodyName>base_link</bodyName>
         <frameId>ardrone_base_link</frameId>
-        <topicName>imu</topicName>
+        <topicName>ardrone/imu</topicName>
         <rpyOffsets>0 0 0</rpyOffsets> <!-- deprecated -->
         <gaussianNoise>0</gaussianNoise>  <!-- deprecated -->
@@ -23,10 +23,10 @@
         <rateGaussianNoise>0.00 0.00 0.00</rateGaussianNoise>
         <headingDrift>0.0</headingDrift>
-      	<headingDriftFrequency>0.0</headingDriftFrequency>
-      	<headingOffset>0.0	</headingOffset>
-      	<rateDriftFrequency>0 0 0</rateDriftFrequency>
-      	<rateOffset>0 0 0</rateOffset>
-      	<accelDriftFrequency>0 0 0</accelDriftFrequency>
-      	<accelOffset>0 0 0</accelOffset>
+	<headingDriftFrequency>0.0</headingDriftFrequency>
+	<headingOffset>0.0	</headingOffset>
+	<rateDriftFrequency>0 0 0</rateDriftFrequency>
+	<rateOffset>0 0 0</rateOffset>
+	<accelDriftFrequency>0 0 0</accelDriftFrequency>
+	<accelOffset>0 0 0</accelOffset>
         <headingGaussianNoise>0.00</headingGaussianNoise>
       </plugin>
@@ -39,5 +39,5 @@
         <offset>0</offset>
         <drift>0.1</drift>
-        <driftFrequency>0.0</driftFrequency>
+	<driftFrequency>0.0</driftFrequency>
         <gaussianNoise>0.5</gaussianNoise>
       </plugin>
@@ -49,5 +49,5 @@
         <offset>0 0 0</offset>
         <drift>0.0 0.0 0.0</drift>
-        <driftFrequency>0.0 0.0 0.0</driftFrequency>
+	<driftFrequency>0.0 0.0 0.0</driftFrequency>
         <gaussianNoise>1.3e-2 1.3e-2 1.3e-2</gaussianNoise>
       </plugin>
@@ -58,12 +58,12 @@
         <topicName>fix</topicName>
         <velocityTopicName>fix_velocity</velocityTopicName>
-      	<offset>0 0 0</offset>
+	<offset>0 0 0</offset>
         <drift>5.0 5.0 5.0</drift>
-      	<driftFrequency>0.0 0.0 0.0</driftFrequency>
+	<driftFrequency>0.0 0.0 0.0</driftFrequency>
         <gaussianNoise>0.1 0.1 0.1</gaussianNoise>
         <velocityDrift>0 0 0</velocityDrift>
         <velocityDriftFrequency>0 0 0</velocityDriftFrequency>
         <velocityGaussianNoise>0.1 0.1 0.1</velocityGaussianNoise>
-      	<velocityOffset>0 0 0</velocityOffset>
+	<velocityOffset>0 0 0</velocityOffset>
       </plugin>
       <plugin name="quadrotor_groundtruth_sim" filename="libgazebo_ros_p3d.so">

File: src/sim_ardrone/src/cvg_sim_gazebo_plugins/urdf/quadrotor_simple_controller.urdf.xacro (robot description, xacro)
@@ -12,5 +12,5 @@
         <bodyName>base_link</bodyName>
         <stateTopic>ground_truth/state</stateTopic>
-        <imuTopic>imu</imuTopic>
+        <imuTopic>ardrone/imu</imuTopic>
         <topicName>cmd_vel</topicName>
         <rollpitchProportionalGain>10.0</rollpitchProportionalGain>
@@ -36,7 +36,7 @@
         <bodyName>base_link</bodyName>
         <stateTopic>ground_truth/state</stateTopic>
-        <imuTopic>imu</imuTopic>
+        <imuTopic>ardrone/imu</imuTopic>
         <sonarTopic>sonar_height</sonarTopic>
-        <lidarTopic>scan</lidarTopic>
+        <lidarTopic>lidar_collision</lidarTopic>
         <topicName>cmd_vel</topicName>
       </plugin>
